File: CESP.kicad_pcb (KiCad board)
At the start: 2 copper layers, 55.9 x 44.7 mm, 9 parts

Commit message: Add initial parts and Snarf Logo
Parts:
- removed the LED-1206 at (201.5, 99.9)
- added CON: USB-Mini-B, USB_MINI_B, F.Cu at (174.0, 99.7)
- added LED-0603: VAL***, LED-0603, F.Cu at (177.8, 121.3)
- added LED-0805: Val*, LED-0805, F.Cu at (177.8, 124.5)
- added LED-1206: VAL**, LED-1206, F.Cu at (162.6, 104.1)
- added LED-1206: VAL**, LED-1206, F.Cu at (178.4, 128.3)
- added MICROSWITCH_SPST: Val**, MICROSWITCH_SPST, F.Cu at (170.2, 134.6)
- added MSOP_8: VAL, MSOP_8, F.Cu at (205.7, 101.6)
- added POT_CMS: Val**, POT_CMS, F.Cu at (171.4, 108.6)
- added PQFP80: VAL***, PQFP80, F.Cu at (198.8, 129.5)
- added SM0603_Capa: Val**, SM0603_Capa, F.Cu at (190.5, 121.3)
- added SOIC24: VAL**, SOIC24, F.Cu at (200.0, 112.4)
- added SOT23: VAL, SOT23, F.Cu at (188.6, 99.1)
- added SOT23: VAL, SOT23, F.Cu at (183.5, 99.1)
- added TQFP32: VAL**, TQFP32, F.Cu at (183.5, 111.1)
- added TSSOP16: Val**, TSSOP16, F.Cu at (195.6, 101.6)
- added VAL: Snarf_mod, Snarf_mod, F.Cu at (179.7, 134.6)
- moved SM0603 38.9 mm to (162.6, 132.1)
- moved TSSOP14 31.9 mm to (172.7, 116.8)
- moved SM0603 25.7 mm to (162.6, 111.8)
- moved SM0603 20.2 mm to (162.6, 109.2)
- moved LED-1206 17.4 mm to (170.2, 124.5)
- moved SOIC24 11.4 mm to (162.6, 121.9)
- moved TSSOP14 2.59 mm to (162.6, 99.1)
